File: hardware/power_input.kicad_sch (KiCad schematic)
At the start: 30 parts, among them J1 Micro-Fit 2x3, J2 Micro-Fit 2x3

Commit message: Layout rev B: top-side two-shunt power stage, 5.0SMDJ60A TVS, crystal by the MCU
Commutation loop 5.0 -> 3.0 nH (FastHenry), 60 V hot-plug peak 106 -> 96 V.
Re-placed and re-routed (Freerouting + tools/hand_route.py); DRC: 0 unconnected,
only the MD80-inherent AUX1/screw courtyard overlap. Docs and sims updated.

Co-Authored-By: Claude Opus 5.5 (1M context) <noreply@anthropic.com>
Parts:
- D1: value SMBJ60A -> 5.0SMDJ60A; footprint Diode_SMD:D_SMB -> Diode_SMD:D_SMC; MPN Littelfuse SMBJ60A -> Littelfuse 5.0SMDJ60A; Note 600 W TVS, VRWM 60 V, VC 96.8 V @ 6.2 A -> 5 kW TVS, VRWM 60 V, VC 96.8 V @ 51.6 A; sized by sim/bus_s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
Changed lines of the file:
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@@
 			)
 		)
-		(property "Value" "SMBJ60A"
+		(property "Value" "5.0SMDJ60A"
 			(at 106.68 36.83 0)
 			(show_name no)
@@
 			)
 		)
-		(property "Footprint" "Diode_SMD:D_SMB"
+		(property "Footprint" "Diode_SMD:D_SMC"
 			(at 106.68 34.29 0)
 			(hide yes)
@@
 			)
 		)
-		(property "MPN" "Littelfuse SMBJ60A"
+		(property "MPN" "Littelfuse 5.0SMDJ60A"
 			(at 106.68 34.29 0)
 			(hide yes)
@@
 			)
 		)
-		(property "Note" "600 W TVS, VRWM 60 V, VC 96.8 V @ 6.2 A"
+		(property "Note" "5 kW TVS, VRWM 60 V, VC 96.8 V @ 51.6 A; sized by sim/bus_surge.py"
 			(at 106.68 34.29 0)
 			(hide yes)
